File: KICAD_FILES/farm_project_first_version/farming_project.kicad_sch (KiCad schematic)
At the start: 17 parts, among them J1 Arduino_MKRWAN_SHIELD, J10 Capteur_temperature_sous_sol, J2 Capteur de pression, J3 Capteur de luminosite, J4 Capteur_de_CO2, J5 Capteur_humidite_sous_sol_10cm, J6 Capteur_humidite_sous_sol_20cm, J7 Capteur_humidite_sous_sol_30cm, J8 DHT22, J9 battery_input

Commit message: deuxieme version PCB
Parts:
- removed C1: 100n, Connector_PinSocket_2.54mm:PinSocket_1x02_P2.54mm_Vertical, symbol Device:C
- removed J5: Capteur_humidite_sous_sol_10cm, Connector_JST:JST_XH_S3B-XH-A-1_1x03_P2.50mm_Horizontal, symbol Connector_Generic:Conn_01x03
- removed J6: Capteur_humidite_sous_sol_20cm, Connector_JST:JST_XH_S3B-XH-A-1_1x03_P2.50mm_Horizontal, symbol Connector_Generic:Conn_01x03
- removed J7: Capteur_humidite_sous_sol_30cm, Connector_JST:JST_XH_S3B-XH-A-1_1x03_P2.50mm_Horizontal, symbol Connector_Generic:Conn_01x03
- added J11: regulateur_tension, Connector_JST:JST_PH_B4B-PH-K_1x04_P2.00mm_Vertical, symbol Connector_Generic:Conn_01x04
- added J5: Capteur_humidite_sous_sol_10cm, Connector_JST:JST_PH_B4B-PH-K_1x04_P2.00mm_Vertical, symbol Connector_Generic:Conn_01x04
- added J6: Capteur_humidite_sous_sol_20cm, Connector_JST:JST_PH_B4B-PH-K_1x04_P2.00mm_Vertical, symbol Connector_Generic:Conn_01x04
- added J7: Capteur_humidite_sous_sol_30cm, Connector_JST:JST_PH_B4B-PH-K_1x04_P2.00mm_Vertical, symbol Connector_Generic:Conn_01x04
- R1, R2: footprint Connector_PinSocket_2.54mm:PinSocket_1x02_P2.54mm_Vertical -> Resistor_THT:R_Axial_DIN0309_L9.0mm_D3.2mm_P12.70mm_Horizontal
Connections:
- net A1: now also J5.4 (Pin_4)
- net A2: now also J6.4 (Pin_4); no longer R1.2, R2.1
- net A3: now also J7.4 (Pin_4)
- net D1: no longer J10.4 (Pin_4)
- net D2: now also J8.4 (Pin_4)
- net D3: no longer J10.3 (Pin_3)
- net D4: no longer J8.4 (Pin_4)
- net D5: now also J10.4 (Pin_4)
- net GND: now also J9.1 (Pin_1), J11.2 (Pin_2), J5.1 (Pin_1), J6.1 (Pin_1), J7.1 (Pin_1); no longer J9.2 (Pin_2)
- net VCC: now also J11.3 (Pin_3); no longer J10.2 (Pin_2), J2.1 (Pin_1), J3.1 (Pin_1), J4.1 (Pin_1), J8.2 (Pin_2)
- net Vbat: now also J9.2 (Pin_2); no longer J9.1 (Pin_1)
- net DAC0/A0 renamed A0
- net A0: now also R1.2, R2.1
- net TX renamed D14
- net D14: now also J11.4 (Pin_4)
- new net VOUT: J10.2 (Pin_2), J11.1 (Pin_1), J2.1 (Pin_1), J3.1 (Pin_1), J4.1 (Pin_1), J5.2 (Pin_2), J6.2 (Pin_2), J7.2 (Pin_2), J8.2 (Pin_2)
- no-connect marks 22 -> 26
Other:
- moved on the sheet: J8

Commit message: mise a jour
Parts:
- J11: footprint Connector_JST:JST_PH_B4B-PH-K_1x04_P2.00mm_Vertical -> Connector_PinHeader_2.54mm:PinHeader_1x04_P2.54mm_Vertical
Changed lines of the file:
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@@
 			)
 		)
-		(property "Footprint" "Connector_JST:JST_PH_B4B-PH-K_1x04_P2.00mm_Vertical"
+		(property "Footprint" "Connector_PinHeader_2.54mm:PinHeader_1x04_P2.54mm_Vertical"
 			(at 246.38 102.87 0)
 			(effects
